Commit message: modified to run on JNano, ESP32 with custom settings

File: linorobot2_description/urdf/2wd_properties.urdf.xacro (robot description, xacro)
@@ -1,22 +1,22 @@
 <?xml version="1.0"?>
 <robot xmlns:xacro="http://ros.org/wiki/xacro">
-  <xacro:property name="base_length" value="0.24" />
-  <xacro:property name="base_width" value="0.275" />
-  <xacro:property name="base_height" value="0.003" />
+  <xacro:property name="base_length" value="0.22" />
+  <xacro:property name="base_width" value="0.18" />
+  <xacro:property name="base_height" value="0.06" />
   <xacro:property name="base_mass" value="1" />
-  <xacro:property name="wheel_radius" value="0.045" />
-  <xacro:property name="wheel_width" value="0.01" />
-  <xacro:property name="wheel_pos_x" value="0.0" />
-  <xacro:property name="wheel_pos_y" value="0.13" />
+  <xacro:property name="wheel_radius" value="0.035" />
+  <xacro:property name="wheel_width" value="0.027" />
+  <xacro:property name="wheel_pos_x" value="-0.07" />
+  <xacro:property name="wheel_pos_y" value="-0.105" />
   <xacro:property name="wheel_pos_z" value="-0.03" />
-  <xacro:property name="wheel_mass" value=".1" />
-  <xacro:property name="wheel_torque" value="20" />
+  <xacro:property name="wheel_mass" value="0.1" />
+  <xacro:property name="wheel_torque" value="10" />
   <xacro:property name="front_caster_wheel" value="true" />
-  <xacro:property name="rear_caster_wheel" value="true" />
+  <xacro:property name="rear_caster_wheel" value="false" />
   <xacro:property name="laser_pose">
-    <origin xyz="0.12 0 0.33" rpy="0 0 0"/>
+    <origin xyz="0.02 0 0.085" rpy="0 -0.0 0"/>
   </xacro:property>
-  <xacro:property name="depth_sensor_pose">
+  <!-- <xacro:property name="depth_sensor_pose">
     <origin xyz="0.14 0.0 0.045" rpy="0 0 0"/>
-  </xacro:property>
+  </xacro:property> -->
 </robot>

File: linorobot2_description/urdf/mech/caster_wheel.urdf.xacro (robot description, xacro)
@@ -4,4 +4,5 @@
     <xacro:property name="caster_wheel_radius" value="${(wheel_radius - wheel_pos_z) / 2}" />
     <xacro:if value="${side == 'front'}">
+        <!--<xacro:property name="caster_wheel_x" value="${(base_length / 2) - (caster_wheel_radius / 4)}" /> -->
         <xacro:property name="caster_wheel_x" value="${(base_length / 2) - caster_wheel_radius}" />
     </xacro:if>

Commit message: added a webcam

File: linorobot2_description/urdf/2wd_properties.urdf.xacro (robot description, xacro)
@@ -17,6 +17,6 @@
     <origin xyz="0.02 0 0.085" rpy="0 -0.0 0"/>
   </xacro:property>
-  <!-- <xacro:property name="depth_sensor_pose">
+  <xacro:property name="webcam_sensor_pose">
     <origin xyz="0.14 0.0 0.045" rpy="0 0 0"/>
-  </xacro:property> -->
+  </xacro:property>
 </robot>

File: linorobot2_description/urdf/robots/2wd.urdf.xacro (robot description, xacro)
@@ -7,4 +7,5 @@
   <xacro:include filename="$(find linorobot2_description)/urdf/sensors/imu.urdf.xacro" />
   <xacro:include filename="$(find linorobot2_description)/urdf/sensors/generic_laser.urdf.xacro" />
+  <xacro:include filename="$(find linorobot2_description)/urdf/sensors/webcam_sensor.urdf.xacro" />
   <xacro:include filename="$(find linorobot2_description)/urdf/sensors/depth_sensor.urdf.xacro" />
   <xacro:include filename="$(find linorobot2_description)/urdf/controllers/diff_drive.urdf.xacro" />
@@ -57,7 +58,7 @@
     <xacro:insert_block name="laser_pose" />
   </xacro:generic_laser>
-  <!-- <xacro:depth_sensor>
-    <xacro:insert_block name="depth_sensor_pose" />
-  </xacro:depth_sensor> -->
+  <xacro:webcam_sensor>
+    <xacro:insert_block name="webcam_sensor_pose" />
+  </xacro:webcam_sensor>
   <xacro:diff_drive_controller
     wheel_separation="${wheel_pos_y * 2}"
