Commit message: Add valid caster contact discriminator
Co-authored-by: Copilot <223556219+Copilot@users.noreply.github.com>

File: linorobot2_description/urdf/mech/caster_wheel.urdf.xacro (robot description, xacro)
@@ -1,5 +1,5 @@
 <?xml version="1.0"?>
 <robot xmlns:xacro="http://ros.org/wiki/xacro">
-  <xacro:macro name="caster_wheel" params="side mass base_length wheel_radius wheel_pos_z">
+  <xacro:macro name="caster_wheel" params="side mass base_length wheel_radius wheel_pos_z caster_mu:=0.01">
     <xacro:property name="caster_wheel_radius" value="${(wheel_radius - wheel_pos_z) / 2}" />
     <xacro:if value="${side == 'front'}">
@@ -35,6 +35,6 @@
     </link>
     <gazebo reference="${side}_caster_wheel_link">
-        <mu1>0.01</mu1>
-        <mu2>0.01</mu2>
+        <mu1>${caster_mu}</mu1>
+        <mu2>${caster_mu}</mu2>
     </gazebo>
     <joint name="${side}_caster_wheel_joint" type="fixed">

File: linorobot2_description/urdf/robots/2wd_fortress.urdf.xacro (robot description, xacro)
@@ -6,4 +6,5 @@
   <xacro:arg name="wheel_mu" default="1.0"/>
   <xacro:arg name="include_caster" default="true"/>
+  <xacro:arg name="caster_mu" default="0.01"/>
   <!-- Geometrieparameter (Pi-Stand / Phase 0 Manifest) -->
   <xacro:property name="base_length" value="0.22" />
@@ -78,4 +79,5 @@
       wheel_radius="${wheel_radius}"
       wheel_pos_z="${wheel_pos_z}"
+      caster_mu="$(arg caster_mu)"
     />
   </xacro:if>
